File: srxe.kicad_pcb (KiCad board)
At the start: 2 copper layers, 48.3 x 10.2 mm, 3 parts

Commit message: align grid
Parts:
- moved H1 9.88 mm to (149.7, 100.0)
- moved U$1 9.88 mm to (135.7, 100.0)
- moved JP2 9.77 mm to (162.5, 100.0)
Other:
- board size 48.3 x 10.2 mm -> 48 x 10 mm

Commit message: mark v0.2
Other:
- board text added: "Smart Response Hacking Group github.com/srhg v0.2 Remix of git.io/SRXE Thanks securelyfitz!"
- board text removed: "Smart Response Hacking Group github.com/srhg Remix of git.io/SRXE Thanks securelyfitz!"
Changed lines of the file:
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@@
   (gr_arc (start 127.25 103.75) (end 126 103.75) (angle -90) (layer Edge.Cuts) (width 0.15))
   (gr_arc (start 127.25 96.25) (end 127.25 95) (angle -90) (layer Edge.Cuts) (width 0.15))
-  (gr_text "Smart Response Hacking Group\ngithub.com/srhg\n\nRemix of git.io/SRXE\nThanks securelyfitz!" (at 172.5289 99.9974) (layer B.SilkS)
+  (gr_text "Smart Response Hacking Group\ngithub.com/srhg\nv0.2\nRemix of git.io/SRXE\nThanks securelyfitz!" (at 172.5289 99.9974) (layer B.SilkS)
     (effects (font (size 1.15 1.15) (thickness 0.2)) (justify left mirror))
   )
